Commit message: feat(curriculum): restructure into 7-week curriculum (Week 0-6) with AI hallucination traps

File: week-4/template_ws/src/apex_simulation/urdf/apex_sim_chassis.urdf.xacro (robot description, xacro)
@@ -1,6 +1,7 @@
 <?xml version="1.0"?>
-<robot xmlns:xacro="http://www.ros.org/wiki/xacro" name="apex_sim_chassis">
-  <!-- ==================== Base Link & Chassis ==================== -->
+<robot xmlns:xacro="http://www.ros.org/wiki/xacro" name="apex_sim_rover">
+  <!-- ==================== Root Kinematic Frame ==================== -->
   <link name="base_link"/>
+  <!-- ==================== Chassis ==================== -->
   <joint name="base_link_to_chassis" type="fixed">
     <parent link="base_link"/>
@@ -10,20 +11,11 @@
   <link name="chassis">
     <visual>
-      <origin xyz="0 0 0" rpy="0 0 0"/>
-      <geometry>
-        <box size="0.6 0.4 0.15"/>
-      </geometry>
-      <material name="dark">
-        <color rgba="0.2 0.2 0.2 1.0"/>
-      </material>
+      <geometry><box size="0.6 0.4 0.15"/></geometry>
+      <material name="dark"><color rgba="0.2 0.2 0.2 1.0"/></material>
     </visual>
     <collision>
-      <origin xyz="0 0 0" rpy="0 0 0"/>
-      <geometry>
-        <box size="0.6 0.4 0.15"/>
-      </geometry>
+      <geometry><box size="0.6 0.4 0.15"/></geometry>
     </collision>
     <inertial>
-      <origin xyz="0 0 0" rpy="0 0 0"/>
       <mass value="15.0"/>
       <inertia ixx="0.22" ixy="0" ixz="0" iyy="0.47" iyz="0" izz="0.65"/>
@@ -40,20 +32,11 @@
     <link name="${name}_link">
       <visual>
-        <origin xyz="0 0 0" rpy="0 0 0"/>
-        <geometry>
-          <cylinder radius="0.1" length="0.06"/>
-        </geometry>
-        <material name="orange">
-          <color rgba="1.0 0.4 0.0 1.0"/>
-        </material>
+        <geometry><cylinder radius="0.1" length="0.06"/></geometry>
+        <material name="orange"><color rgba="1.0 0.4 0.0 1.0"/></material>
       </visual>
       <collision>
-        <origin xyz="0 0 0" rpy="0 0 0"/>
-        <geometry>
-          <cylinder radius="0.1" length="0.06"/>
-        </geometry>
+        <geometry><cylinder radius="0.1" length="0.06"/></geometry>
       </collision>
       <inertial>
-        <origin xyz="0 0 0" rpy="0 0 0"/>
         <mass value="1.5"/>
         <inertia ixx="0.004" ixy="0" ixz="0" iyy="0.004" iyz="0" izz="0.0075"/>
@@ -78,17 +61,9 @@
   <link name="lidar_link">
     <visual>
-      <origin xyz="0 0 0" rpy="0 0 0"/>
-      <geometry>
-        <cylinder radius="0.05" length="0.06"/>
-      </geometry>
-      <material name="blue">
-        <color rgba="0.1 0.3 0.9 1.0"/>
-      </material>
+      <geometry><cylinder radius="0.05" length="0.06"/></geometry>
+      <material name="blue"><color rgba="0.1 0.3 0.9 1.0"/></material>
     </visual>
     <collision>
-      <origin xyz="0 0 0" rpy="0 0 0"/>
-      <geometry>
-        <cylinder radius="0.05" length="0.06"/>
-      </geometry>
+      <geometry><cylinder radius="0.05" length="0.06"/></geometry>
     </collision>
     <inertial>
@@ -97,6 +72,25 @@
     </inertial>
   </link>
+  <!-- ==================== Front Camera ==================== -->
+  <joint name="camera_joint" type="fixed">
+    <parent link="chassis"/>
+    <child link="camera_link"/>
+    <origin xyz="0.30 0 0.05" rpy="0 0 0"/>
+  </joint>
+  <link name="camera_link">
+    <visual>
+      <geometry><box size="0.04 0.12 0.03"/></geometry>
+      <material name="silver"><color rgba="0.7 0.7 0.7 1.0"/></material>
+    </visual>
+    <collision>
+      <geometry><box size="0.04 0.12 0.03"/></geometry>
+    </collision>
+    <inertial>
+      <mass value="0.1"/>
+      <inertia ixx="0.0001" ixy="0" ixz="0" iyy="0.0001" iyz="0" izz="0.0001"/>
+    </inertial>
+  </link>
   <!-- ==================== Gazebo Plugins ==================== -->
-  <!-- Differential Drive Motor Controller -->
+  <!-- 1. Differential Drive Motor Controller -->
   <gazebo>
     <plugin name="diff_drive" filename="libgazebo_ros_diff_drive.so">
@@ -104,5 +98,5 @@
         <namespace>/</namespace>
         <remapping>cmd_vel:=cmd_vel</remapping>
-        <remapping>odom:=wheel/odom</remapping>
+        <remapping>odom:=odom</remapping>
       </ros>
       <left_joint>rear_left_wheel_joint</left_joint>
@@ -111,5 +105,4 @@
       <wheel_diameter>0.20</wheel_diameter>
       <max_wheel_torque>20.0</max_wheel_torque>
-      <max_wheel_acceleration>2.0</max_wheel_acceleration>
       <publish_odom>true</publish_odom>
       <publish_odom_tf>true</publish_odom_tf>
@@ -118,10 +111,10 @@
     </plugin>
   </gazebo>
-  <!-- 2D LiDAR Ray Sensor -->
+  <!-- 2. LiDAR Ray Sensor -->
   <gazebo reference="lidar_link">
     <sensor name="lidar_sensor" type="ray">
       <always_on>true</always_on>
       <update_rate>10.0</update_rate>
-      <visualize>true</visualize>
+      <visualize>false</visualize>
       <ray>
         <scan>
@@ -135,6 +128,5 @@
         <range>
           <min>0.15</min>
-          <max>12.0</max>
-          <resolution>0.01</resolution>
+          <max>10.0</max>
         </range>
       </ray>
@@ -148,3 +140,30 @@
     </sensor>
   </gazebo>
+  <!-- 3. Front Camera Sensor -->
+  <gazebo reference="camera_link">
+    <sensor name="front_camera" type="camera">
+      <always_on>true</always_on>
+      <update_rate>20.0</update_rate>
+      <camera>
+        <horizontal_fov>1.089</horizontal_fov>
+        <image>
+          <width>640</width>
+          <height>480</height>
+          <format>R8G8B8</format>
+        </image>
+        <clip>
+          <near>0.05</near>
+          <far>50.0</far>
+        </clip>
+      </camera>
+      <plugin name="gazebo_camera" filename="libgazebo_ros_camera.so">
+        <ros>
+          <remapping>~/image_raw:=camera/image_raw</remapping>
+          <remapping>~/camera_info:=camera/camera_info</remapping>
+        </ros>
+        <camera_name>camera</camera_name>
+        <frame_name>camera_link</frame_name>
+      </plugin>
+    </sensor>
+  </gazebo>
 </robot>
